File: hardware/BomberCat.kicad_sch (KiCad schematic)
At the start: 86 parts, among them J1 Battery, J3 MAGSPOOF, P1 USB_C_Plug_USB2.0, Q1 DMG3415U-7, SW1 RESET, SW2 GPIO, SW3 ON, SW4 SOURCE MAG, U1 PN7150B0HN_C11002E-PN7150B0HN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, U2 RP2040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

Commit message: update 12Mhz cristal part number
Parts:
- Y2: LCSC# C709001 -> (none); manf# (none) -> 445I23D12M00000; provedor LCSC -> MOUSER
Changed lines of the file:
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@@
       (effects (font (size 1.27 1.27)) hide)
     )
-    (property "manf#" "" (at 26.924 163.449 0)
+    (property "manf#" "445I23D12M00000" (at 26.924 163.449 0)
       (effects (font (size 1.27 1.27)) hide)
     )
-    (property "provedor" "LCSC" (at 26.924 163.449 0)
+    (property "provedor" "MOUSER" (at 26.924 163.449 0)
       (effects (font (size 1.27 1.27)) hide)
     )
-    (property "LCSC#" "C709001" (at 26.924 163.449 0)
+    (property "LCSC#" "" (at 26.924 163.449 0)
       (effects (font (size 1.27 1.27)) hide)
     )

Commit message: feat(hw): add Embedded Antenna
Parts:
- added J4: MAGSPOOF, Connector_PinHeader_2.54mm:PinHeader_1x02_P2.54mm_Vertical, symbol Connector_Generic:Conn_01x02
- added L4: 30t_30mm, BomberCat:Coil_30t_30mm_0.2_0.2_0.6_0.3, symbol Magspoof:Coil_20t_35mm_0.2_0.6_0.3
- J3: now not fitted
Connections:
- net OUTA: now also J4.1 (Pin_1), L4.1
- net OUTB: now also J4.2 (Pin_2), L4.2

Commit message: fix(hw): update part numbers
Parts:
- C5: LCSC# C15849 -> C5673; manf# (none) -> CL10A105KA8NNNC
- C6, C8: LCSC# C15849 -> C5673
- P1: LCSC# C2987386 -> C393939
- R1, R2: LCSC# C169849 -> C2930027; manf# ERJ3GEYJ103V -> FRC0603J103 TS
- R4, R5: LCSC# C191782 -> C122969; manf# ERJ3RBD5101V -> RT0603BRD075K1L
- R6, R7: manf# WR06X104JTL -> 0603WAJ0104T5E
- U1: LCSC# C11002 -> C702907; manf# PN7150B0HN -> PN7150B0HN/C11002E
- U3: value MCP73831-3-OT -> MCP73831T-2DCI/OT; manf# MCP73831-3-OT -> MCP73831T-2DCI/OT
Other:
- note added: "Charge at 196mA"
- moved on the sheet: C6, C7, C8, C9

Commit message: fix (hw): Update part numbers
Parts:
- C23: manf# (none) -> CC0603KRX7R7BB102; provedor MOUSER -> LCSC
- C29: LCSC# C85713 -> C96446; manf# (none) -> CL10A106MA8NRNC
- C30, C31: LCSC# C561174 -> C107035; manf# C0603C121J5GAC -> CC0603JRNPO9BN121
- C34: LCSC# C466781 -> C96446; manf# C0603X5R106M160NT -> CL10A106MA8NRNC
- J1: now not fitted
- JP1: now not fitted; now left out of the parts list
- L3: manf# CONUFL001-SMD -> CONUFL001-SMD-T
- R17, R20: LCSC# C169849 -> C2930027; manf# ERJ3GEYJ103V -> FRC0603J103 TS
- SW1, SW2: LCSC# C2886897 -> C318889
- U5: manf# ESP32-WROOM-32D -> ESP32M4
Other:
- note added: "GREEN"
Changed lines of the file:
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@@
 		(comment 1 "Andres Sabas")
 	)
+	(text "GREEN"
+		(exclude_from_sim no)
+		(at 172.466 64.516 0)
+		(effects
+			(font
+				(size 1.27 1.27)
+			)
+		)
+	)
 	(text "COIL"
 		(exclude_from_sim no)
@@
 		)
 	)
+	(text "GREEN"
+		(exclude_from_sim no)
+		(at 139.192 268.732 0)
+		(effects
+			(font
+				(size 1.27 1.27)
+			)
+		)
+	)
 	(text "LEDS & BUTTONS"
 		(exclude_from_sim no)
@@
 		)
 	)
+	(text "GREEN"
+		(exclude_from_sim no)
+		(at 172.466 82.042 0)
+		(effects
+			(font
+				(size 1.27 1.27)
+			)
+		)
+	)
 	(text "WIFI & BLE NINA"
 		(exclude_from_sim no)
@@
 			)
 		)
-		(property "manf#" "ESP32-WROOM-32D"
+		(property "manf#" "ESP32M4"
 			(at 238.506 153.416 0)
 			(effects
@@
 		(in_bom yes)
 		(on_board yes)
-		(dnp no)
+		(dnp yes)
 		(property "Reference" "J1"
 			(at 164.084 250.3932 0)
@@
 			)
 		)
-		(property "LCSC#" "C169849"
+		(property "LCSC#" "C2930027"
 			(at 340.614 41.656 0)
 			(effects
@@
 			)
 		)
-		(property "manf#" "ERJ3GEYJ103V"
+		(property "manf#" "FRC0603J103 TS"
 			(at 340.614 41.656 0)
 			(effects
@@
 			)
 		)
-		(property "LCSC#" "C466781"
+		(property "LCSC#" "C96446"
 			(at 381.127 152.654 0)
 			(effects
@@
 			)
 		)
-		(property "manf#" "C0603X5R106M160NT"
+		(property "manf#" "CL10A106MA8NRNC"
 			(at 381.127 152.654 0)
 			(effects
@@
 			)
 		)
-		(property "manf#" "C0603C121J5GAC"
+		(property "manf#" "CC0603JRNPO9BN121"
 			(at 231.902 54.737 0)
 			(effects
@@
 			)
 		)
-		(property "LCSC#" "C561174"
+		(property "LCSC#" "C107035"
 			(at 231.902 54.737 0)
 			(effects
@@
 			)
 		)
-		(property "LCSC#" "C169849"
+		(property "LCSC#" "C2930027"
 			(at 222.25 115.189 0)
 			(effects
@@
 			)
 		)
-		(property "manf#" "ERJ3GEYJ103V"
+		(property "manf#" "FRC0603J103 TS"
 			(at 222.25 115.189 0)
 			(effects
@@
 			)
 		)
-		(property "LCSC#" "C2886897"
+		(property "LCSC#" "C318889"
 			(at 171.069 43.434 0)
 			(effects
@@
 			)
 		)
-		(property "manf#" "CONUFL001-SMD"
+		(property "manf#" "CONUFL001-SMD-T "
 			(at 256.032 50.673 0)
 			(effects
@@
 			)
 		)
-		(property "manf#" ""
+		(property "manf#" "CC0603KRX7R7BB102"
 			(at 213.487 30.353 0)
 			(effects
@@
 			)
 		)
-		(property "provedor" "MOUSER"
+		(property "provedor" "LCSC"
 			(at 213.487 30.353 0)
 			(effects
@@
 		(unit 1)
 		(exclude_from_sim no)
-		(in_bom yes)
+		(in_bom no)
 		(on_board yes)
-		(dnp no)
+		(dnp yes)
 		(fields_autoplaced yes)
 		(property "Reference" "JP1"
@@
 			)
 		)
-		(property "manf#" ""
+		(property "manf#" "CL10A106MA8NRNC"
 			(at 230.632 254 0)
 			(effects
@@
 			)
 		)
-		(property "LCSC#" "C85713"
+		(property "LCSC#" "C96446"
 			(at 230.632 254 0)
 			(effects
@@
 			)
 		)
-		(property "manf#" "C0603C121J5GAC"
+		(property "manf#" "CC0603JRNPO9BN121"
 			(at 231.902 46.99 0)
 			(effects
@@
 			)
 		)
-		(property "LCSC#" "C561174"
+		(property "LCSC#" "C107035"
 			(at 231.902 46.99 0)
 			(effects
@@
 			)
 		)
-		(property "LCSC#" "C2886897"
+		(property "LCSC#" "C318889"
 			(at 171.069 29.718 0)
 			(effects

Commit message: fix(hw): Update LCSC part numbers in schematic
Updates the LCSC part numbers in the schematic to ensure their availability
Parts:
- R4, R5: LCSC# C122969 -> C23186
- U7: LCSC# C636876 -> C44150
Changed lines of the file:
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@@
 			)
 		)
-		(property "LCSC#" "C122969"
+		(property "LCSC#" "C23186"
 			(at 49.784 241.046 0)
 			(effects
@@
 			)
 		)
-		(property "LCSC#" "C636876"
+		(property "LCSC#" "C44150"
 			(at 360.807 146.939 0)
 			(effects
@@
 			)
 		)
-		(property "LCSC#" "C122969"
+		(property "LCSC#" "C23186"
 			(at 49.784 238.506 0)
 			(effects

Commit message: fix(hw): update BOM
Parts:
- H1, H2, H3, H4: now not fitted
- P1: manf# TYPE-C-31-M-31 -> (none)
- R1, R17, R2, R20: manf# FRC0603J103 TS -> (none)
- R14, R21, R22: manf# WR06X104JTL -> (none)
- R6, R7: manf# 0603WAJ0104T5E -> (none)
- R8: value 5.1K -> 5k1; LCSC# C73801 -> C23186
Connections:
- net at D4.1 (K), Q1.2 (S): now also SW3.2 (B); no longer SW3.1 (A)
- net at C22.1, U4.1 (VIN), U4.3 (EN): now also SW3.1 (A); no longer SW3.2 (B)
Changed lines of the file:
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@@
 		(lib_id "Switch:SW_SPST")
 		(at 197.485 251.46 0)
+		(mirror y)
 		(unit 1)
 		(exclude_from_sim no)
@@
 			)
 		)
-		(property "manf#" "FRC0603J103 TS"
+		(property "manf#" ""
 			(at 28.067 37.211 0)
 			(effects
@@
 		(in_bom yes)
 		(on_board yes)
-		(dnp no)
+		(dnp yes)
 		(property "Reference" "H1"
 			(at 272.796 262.4836 0)
@@
 		(in_bom yes)
 		(on_board yes)
-		(dnp no)
+		(dnp yes)
 		(property "Reference" "H4"
 			(at 272.923 277.5966 0)
@@
 			)
 		)
-		(property "manf#" "FRC0603J103 TS"
+		(property "manf#" ""
 			(at 340.614 41.656 0)
 			(effects
@@
 			)
 		)
-		(property "manf#" "WR06X104JTL"
+		(property "manf#" ""
 			(at 350.647 235.712 0)
 			(effects
@@
 			)
 		)
-		(property "manf#" "FRC0603J103 TS"
+		(property "manf#" ""
 			(at 22.225 37.338 0)
 			(effects
@@
 			)
 		)
-		(property "manf#" "0603WAJ0104T5E"
+		(property "manf#" ""
 			(at 88.138 245.1354 0)
 			(effects
@@
 			)
 		)
-		(property "manf#" "FRC0603J103 TS"
+		(property "manf#" ""
 			(at 222.25 115.189 0)
 			(effects
@@
 			)
 		)
-		(property "Value" "5.1K"
+		(property "Value" "5k1"
 			(at 108.839 250.825 90)
 			(effects
@@
 			)
 		)
-		(property "LCSC#" "C73801"
+		(property "LCSC#" "C23186"
 			(at 108.839 253.492 0)
 			(effects
@@
 			)
 		)
-		(property "manf#" "0603WAJ0104T5E"
+		(property "manf#" ""
 			(at 88.138 251.968 0)
 			(effects
@@
 			)
 		)
-		(property "manf#" "TYPE-C-31-M-31"
+		(property "manf#" ""
 			(at 30.226 248.666 0)
 			(effects
@@
 			)
 		)
-		(property "manf#" "WR06X104JTL"
+		(property "manf#" ""
 			(at 177.292 258.191 0)
 			(effects
@@
 		(in_bom yes)
 		(on_board yes)
-		(dnp no)
+		(dnp yes)
 		(property "Reference" "H2"
 			(at 272.796 267.5636 0)
@@
 			)
 		)
-		(property "manf#" "WR06X104JTL"
+		(property "manf#" ""
 			(at 370.713 235.585 0)
 			(effects
@@
 		(in_bom yes)
 		(on_board yes)
-		(dnp no)
+		(dnp yes)
 		(property "Reference" "H3"
 			(at 272.923 272.5166 0)

Commit message: fix(hw): update manf#s
Parts:
- C23: manf# CC0603KRX7R7BB102 -> (none)
- C5: manf# CL10A105KA8NNNC -> (none)
- R4, R5: manf# RT0603BRD075K1L -> (none)
- R8: manf# RS-03K512KT -> (none)
Changed lines of the file:
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@@
 			)
 		)
-		(property "manf#" "RT0603BRD075K1L"
+		(property "manf#" ""
 			(at 49.784 241.046 0)
 			(effects
@@
 			)
 		)
-		(property "manf#" "CC0603KRX7R7BB102"
+		(property "manf#" ""
 			(at 213.487 30.353 0)
 			(effects
@@
 			)
 		)
-		(property "manf#" "RS-03K512KT"
+		(property "manf#" ""
 			(at 108.839 253.492 0)
 			(effects
@@
 			)
 		)
-		(property "manf#" "RT0603BRD075K1L"
+		(property "manf#" ""
 			(at 49.784 238.506 0)
 			(effects
@@
 			)
 		)
-		(property "manf#" "CL10A105KA8NNNC"
+		(property "manf#" ""
 			(at 96.393 25.527 0)
 			(effects

Commit message: fix(hw): add alternative part number of battery charger
Parts:
- U3: LCSC# - -> C424093; Proveedor2 (none) -> JLCPCB
Changed lines of the file:
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@@
 			)
 		)
-		(property "LCSC#" "-"
+		(property "LCSC#" "C424093"
 			(at 123.19 250.952 0)
 			(effects
+				(font
+					(size 1.27 1.27)
+				)
+				(hide yes)
+			)
+		)
+		(property "Proveedor2" "JLCPCB"
+			(at 123.19 250.952 0)
+			(effects
